Commit message: add airbot

File: openteach/components/environment/assets/urdf/allegro_hand_description/urdf/table.urdf (robot description, URDF)
Before this commit: robot table, 2 links, 1 joints
Links:
- link robot_stand: geometry collision box size=0.25 0.25 0.05; visual mesh filename=../meshes/table/table.obj
